File: beduino_kw41z/beduino_kw41z_panel.kicad_pcb (KiCad board)
At the start: 2 copper layers, 83 x 100 mm, 328 parts, among them J1 USB_OTG, J2 Conn_01x07, J3 Conn_01x07, Q1 Q_PMOS_GSD, SW1 SW_Push, SW2 Reset, U1 TC1017, U2 LPC11U35FHI33-501, U3 TC1017, U4 Module_CONN, U5 MKW41Z, Y1 12MHz, Y2 32MHz, Y3 32KHz

Commit message: Remove unused stuff.
Parts:
- removed the C1 at (32.1, 95.8)
- removed the C1 at (32.1, 74.8)
- removed the C1 at (32.1, 53.8)
- removed the C12 at (60.8, 102.2)
- removed the C12 at (60.8, 81.2)
- removed the C12 at (60.8, 60.2)
- removed the C4 at (36.5, 99.2)
- removed the C4 at (36.5, 78.2)
- removed the C4 at (36.5, 57.2)
- removed the C5 at (45.2, 95.5)
- removed the C5 at (45.2, 74.5)
- removed the C5 at (45.2, 53.5)
- removed the C7 at (42.2, 95.5)
- removed the C7 at (42.2, 74.5)
- removed the C7 at (42.2, 53.5)
- removed the C9 at (60.8, 99.0)
- removed the C9 at (60.8, 78.0)
- removed the C9 at (60.8, 57.0)
- removed the D1 at (38.5, 95.8)
- removed the D1 at (38.5, 74.8)
- removed the D1 at (38.5, 53.8)
- removed the D2 at (40.2, 109.7)
- removed the D2 at (40.2, 88.7)
- removed the D2 at (40.2, 67.7)
- removed the D3 at (43.8, 109.7)
- removed the D3 at (43.8, 88.7)
- removed the D3 at (43.8, 67.7)
- removed the D4 at (47.2, 109.7)
- removed the D4 at (47.2, 88.7)
- removed the D4 at (47.2, 67.7)
- removed the D5 at (63.2, 105.5)
- removed the D5 at (63.2, 84.5)
- removed the D5 at (63.2, 63.5)
- removed the D6 at (63.2, 97.1)
- removed the D6 at (63.2, 76.1)
- removed the D6 at (63.2, 55.1)
- removed the D7 at (58.0, 102.2)
- removed the D7 at (58.0, 81.2)
- removed the D7 at (58.0, 60.2)
- removed the D8 at (58.0, 104.2)
- removed the D8 at (58.0, 83.2)
- removed the D8 at (58.0, 62.2)
- removed the L1 at (84.8, 106.0)
- removed the L1 at (84.8, 85.0)
- removed the L1 at (84.8, 64.0)
- removed the Q1 at (37.8, 109.3)
- removed the Q1 at (37.8, 88.3)
- removed the Q1 at (37.8, 67.3)
- removed the R1 at (37.8, 103.8)
- removed the R1 at (37.8, 82.8)
- removed the R1 at (37.8, 61.8)
- removed the R10 at (48.5, 101.2)
- removed the R10 at (48.5, 80.2)
- removed the R10 at (48.5, 59.2)
- removed the R11 at (48.5, 103.0)
- removed the R11 at (48.5, 82.0)
- removed the R11 at (48.5, 61.0)
- removed the R13 at (48.5, 106.5)
- removed the R13 at (48.5, 85.5)
- removed the R13 at (48.5, 64.5)
- removed the R13-R10 at (48.5, 104.8)
- removed the R13-R10 at (48.5, 83.8)
- removed the R13-R10 at (48.5, 62.8)
- removed the R13-R10 at (48.5, 41.8)
- removed the R14 at (66.5, 105.5)
- removed the R14 at (66.5, 84.5)
- removed the R14 at (66.5, 63.5)
- removed the R15 at (66.5, 97.1)
- removed the R15 at (66.5, 76.1)
- removed the R15 at (66.5, 55.1)
- removed the R16 at (63.6, 99.5)
- removed the R16 at (63.6, 78.5)
- removed the R16 at (63.6, 57.5)
- removed the R2 at (37.8, 102.2)
- removed the R2 at (37.8, 81.2)
- removed the R2 at (37.8, 60.2)
- removed the R2 at (37.8, 39.2)
- removed the R3 at (37.8, 106.0)
- removed the R3 at (37.8, 85.0)
- removed the R3 at (37.8, 64.0)
- removed the R4 at (38.2, 100.0)
- removed the R4 at (38.2, 79.0)
- removed the R4 at (38.2, 58.0)
- removed the R5 at (48.5, 99.5)
- removed the R5 at (48.5, 78.5)
- removed the R5 at (48.5, 57.5)
- removed the R6 at (42.0, 109.7)
- removed the R6 at (42.0, 88.7)
- removed the R6 at (42.0, 67.7)
- removed the R7 at (45.5, 109.7)
- removed the R7 at (45.5, 88.7)
- removed the R7 at (45.5, 67.7)
- removed the R8 at (49.0, 109.7)
- removed the R8 at (49.0, 88.7)
- removed the R8 at (49.0, 67.7)
- removed the R8 at (49.0, 46.6)
- removed the R9 at (48.6, 95.5)
- removed the R9 at (48.6, 74.5)
- removed the R9 at (48.6, 53.5)
- removed the SW1 at (33.2, 109.2)
- removed the SW1 at (33.2, 88.2)
- removed the SW1 at (33.2, 67.2)
- removed the SW2 at (64.5, 102.5)
- removed the SW2 at (64.5, 81.5)
- removed the SW2 at (64.5, 60.5)
- removed the U1 at (35.0, 95.8)
- removed the U1 at (35.0, 74.8)
- removed the U1 at (35.0, 53.8)
- removed the U2 at (43.2, 103.8)
- removed the U2 at (43.2, 82.8)
- removed the U2 at (43.2, 61.8)
- removed the U3 at (58.0, 99.0)
- removed the U3 at (58.0, 78.0)
- removed the U3 at (58.0, 57.0)
- removed the U5 at (79.5, 102.5)
- removed the U5 at (79.5, 81.5)
- removed the U5 at (79.5, 60.5)
- removed the Y1 at (44.0, 98.0)
- removed the Y1 at (44.0, 77.0)
- removed the Y1 at (44.0, 56.0)
- removed the Y2 at (82.6, 107.7)
- removed the Y2 at (82.6, 86.7)
- removed the Y2 at (82.6, 65.7)
- removed the Y3 at (76.5, 107.5)
- removed the Y3 at (76.5, 86.5)
- removed the Y3 at (76.5, 65.5)
- removed the Y3 at (76.5, 44.5)
- added C1: 1u, Capacitor_SMD:C_0603_1608Metric, F.Cu at (32.1, 95.8)
- added C1: 1u, Capacitor_SMD:C_0603_1608Metric, F.Cu at (32.1, 74.8)
- added C1: 1u, Capacitor_SMD:C_0603_1608Metric, F.Cu at (32.1, 53.8)
- added C12: 10u, Capacitor_SMD:C_0603_1608Metric, F.Cu at (60.8, 102.2)
- added C12: 10u, Capacitor_SMD:C_0603_1608Metric, F.Cu at (60.8, 81.2)
- added C12: 10u, Capacitor_SMD:C_0603_1608Metric, F.Cu at (60.8, 60.2)
- added C4: 10u, Capacitor_SMD:C_0603_1608Metric, F.Cu at (36.5, 99.2)
- added C4: 10u, Capacitor_SMD:C_0603_1608Metric, F.Cu at (36.5, 78.2)
- added C4: 10u, Capacitor_SMD:C_0603_1608Metric, F.Cu at (36.5, 57.2)
- added C5: 18p, Capacitor_SMD:C_0603_1608Metric, F.Cu at (45.2, 95.5)
- added C5: 18p, Capacitor_SMD:C_0603_1608Metric, F.Cu at (45.2, 74.5)
- added C5: 18p, Capacitor_SMD:C_0603_1608Metric, F.Cu at (45.2, 53.5)
- added C7: 18p, Capacitor_SMD:C_0603_1608Metric, F.Cu at (42.2, 95.5)
- added C7: 18p, Capacitor_SMD:C_0603_1608Metric, F.Cu at (42.2, 74.5)
- added C7: 18p, Capacitor_SMD:C_0603_1608Metric, F.Cu at (42.2, 53.5)
- added C9: 1u, Capacitor_SMD:C_0603_1608Metric, F.Cu at (60.8, 99.0)
- added C9: 1u, Capacitor_SMD:C_0603_1608Metric, F.Cu at (60.8, 78.0)
- added C9: 1u, Capacitor_SMD:C_0603_1608Metric, F.Cu at (60.8, 57.0)
- added D1: BAT60A, Diode_SMD:D_SOD-323, F.Cu at (38.5, 95.8)
- added D1: BAT60A, Diode_SMD:D_SOD-323, F.Cu at (38.5, 74.8)
- added D1: BAT60A, Diode_SMD:D_SOD-323, F.Cu at (38.5, 53.8)
- added D2: Red, LED_SMD:LED_0603_1608Metric, F.Cu at (40.2, 109.7)
- added D2: Red, LED_SMD:LED_0603_1608Metric, F.Cu at (40.2, 88.7)
- added D2: Red, LED_SMD:LED_0603_1608Metric, F.Cu at (40.2, 67.7)
- added D3: Yellow, LED_SMD:LED_0603_1608Metric, F.Cu at (43.8, 109.7)
- added D3: Yellow, LED_SMD:LED_0603_1608Metric, F.Cu at (43.8, 88.7)
- added D3: Yellow, LED_SMD:LED_0603_1608Metric, F.Cu at (43.8, 67.7)
- added D4: Green, LED_SMD:LED_0603_1608Metric, F.Cu at (47.2, 109.7)
- added D4: Green, LED_SMD:LED_0603_1608Metric, F.Cu at (47.2, 88.7)
- added D4: Green, LED_SMD:LED_0603_1608Metric, F.Cu at (47.2, 67.7)
- added D5: Red, LED_SMD:LED_0603_1608Metric, F.Cu at (63.2, 105.5)
- added D5: Red, LED_SMD:LED_0603_1608Metric, F.Cu at (63.2, 84.5)
- added D5: Red, LED_SMD:LED_0603_1608Metric, F.Cu at (63.2, 63.5)
- added D6: Green, LED_SMD:LED_0603_1608Metric, F.Cu at (63.2, 97.1)
- added D6: Green, LED_SMD:LED_0603_1608Metric, F.Cu at (63.2, 76.1)
- added D6: Green, LED_SMD:LED_0603_1608Metric, F.Cu at (63.2, 55.1)
- added D7: BAT60A, Diode_SMD:D_SOD-323, F.Cu at (58.0, 102.2)
- added D7: BAT60A, Diode_SMD:D_SOD-323, F.Cu at (58.0, 81.2)
- added D7: BAT60A, Diode_SMD:D_SOD-323, F.Cu at (58.0, 60.2)
- added D8: BAT60A, Diode_SMD:D_SOD-323, F.Cu at (58.0, 104.2)
- added D8: BAT60A, Diode_SMD:D_SOD-323, F.Cu at (58.0, 83.2)
- added D8: BAT60A, Diode_SMD:D_SOD-323, F.Cu at (58.0, 62.2)
- added L1: 5.1n, Inductor_SMD:L_0402_1005Metric, F.Cu at (84.8, 106.0)
- added L1: 5.1n, Inductor_SMD:L_0402_1005Metric, F.Cu at (84.8, 85.0)
- added L1: 5.1n, Inductor_SMD:L_0402_1005Metric, F.Cu at (84.8, 64.0)
- added Q1: Q_PMOS_GSD, Package_TO_SOT_SMD:SOT-23, F.Cu at (37.8, 109.3)
- added Q1: Q_PMOS_GSD, Package_TO_SOT_SMD:SOT-23, F.Cu at (37.8, 88.3)
- added Q1: Q_PMOS_GSD, Package_TO_SOT_SMD:SOT-23, F.Cu at (37.8, 67.3)
- added R1: 33, Resistor_SMD:R_0603_1608Metric, F.Cu at (37.8, 103.8)
- added R1: 33, Resistor_SMD:R_0603_1608Metric, F.Cu at (37.8, 82.8)
- added R1: 33, Resistor_SMD:R_0603_1608Metric, F.Cu at (37.8, 61.8)
- added R10: 470, Resistor_SMD:R_0603_1608Metric, F.Cu at (48.5, 101.2)
- added R10: 470, Resistor_SMD:R_0603_1608Metric, F.Cu at (48.5, 80.2)
- added R10: 470, Resistor_SMD:R_0603_1608Metric, F.Cu at (48.5, 59.2)
- added R11: 470, Resistor_SMD:R_0603_1608Metric, F.Cu at (48.5, 103.0)
- added R11: 470, Resistor_SMD:R_0603_1608Metric, F.Cu at (48.5, 82.0)
- added R11: 470, Resistor_SMD:R_0603_1608Metric, F.Cu at (48.5, 61.0)
- added R13: 470, Resistor_SMD:R_0603_1608Metric, F.Cu at (48.5, 106.5)
- added R13: 470, Resistor_SMD:R_0603_1608Metric, F.Cu at (48.5, 85.5)
- added R13: 470, Resistor_SMD:R_0603_1608Metric, F.Cu at (48.5, 64.5)
- added R13-R10: 470, Resistor_SMD:R_0603_1608Metric, F.Cu at (48.5, 104.8)
- added R13-R10: 470, Resistor_SMD:R_0603_1608Metric, F.Cu at (48.5, 83.8)
- added R13-R10: 470, Resistor_SMD:R_0603_1608Metric, F.Cu at (48.5, 62.8)
- added R13-R10: 470, Resistor_SMD:R_0603_1608Metric, F.Cu at (48.5, 41.8)
- added R14: 470, Resistor_SMD:R_0603_1608Metric, F.Cu at (66.5, 105.5)
- added R14: 470, Resistor_SMD:R_0603_1608Metric, F.Cu at (66.5, 84.5)
- added R14: 470, Resistor_SMD:R_0603_1608Metric, F.Cu at (66.5, 63.5)
- added R15: 470, Resistor_SMD:R_0603_1608Metric, F.Cu at (66.5, 97.1)
- added R15: 470, Resistor_SMD:R_0603_1608Metric, F.Cu at (66.5, 76.1)
- added R15: 470, Resistor_SMD:R_0603_1608Metric, F.Cu at (66.5, 55.1)
- added R16: 10k, Resistor_SMD:R_0603_1608Metric, F.Cu at (63.6, 99.5)
- added R16: 10k, Resistor_SMD:R_0603_1608Metric, F.Cu at (63.6, 78.5)
- added R16: 10k, Resistor_SMD:R_0603_1608Metric, F.Cu at (63.6, 57.5)
- added R2: 33, Resistor_SMD:R_0603_1608Metric, F.Cu at (37.8, 102.2)
- added R2: 33, Resistor_SMD:R_0603_1608Metric, F.Cu at (37.8, 81.2)
- added R2: 33, Resistor_SMD:R_0603_1608Metric, F.Cu at (37.8, 60.2)
- added R2: 33, Resistor_SMD:R_0603_1608Metric, F.Cu at (37.8, 39.2)
- added R3: 1k5, Resistor_SMD:R_0603_1608Metric, F.Cu at (37.8, 106.0)
- added R3: 1k5, Resistor_SMD:R_0603_1608Metric, F.Cu at (37.8, 85.0)
- added R3: 1k5, Resistor_SMD:R_0603_1608Metric, F.Cu at (37.8, 64.0)
- added R4: 10k, Resistor_SMD:R_0603_1608Metric, F.Cu at (38.2, 100.0)
- added R4: 10k, Resistor_SMD:R_0603_1608Metric, F.Cu at (38.2, 79.0)
- added R4: 10k, Resistor_SMD:R_0603_1608Metric, F.Cu at (38.2, 58.0)
- added R5: 10k, Resistor_SMD:R_0603_1608Metric, F.Cu at (48.5, 99.5)
- added R5: 10k, Resistor_SMD:R_0603_1608Metric, F.Cu at (48.5, 78.5)
- added R5: 10k, Resistor_SMD:R_0603_1608Metric, F.Cu at (48.5, 57.5)
- added R6: 470, Resistor_SMD:R_0603_1608Metric, F.Cu at (42.0, 109.7)
- added R6: 470, Resistor_SMD:R_0603_1608Metric, F.Cu at (42.0, 88.7)
- added R6: 470, Resistor_SMD:R_0603_1608Metric, F.Cu at (42.0, 67.7)
- added R7: 470, Resistor_SMD:R_0603_1608Metric, F.Cu at (45.5, 109.7)
- added R7: 470, Resistor_SMD:R_0603_1608Metric, F.Cu at (45.5, 88.7)
- added R7: 470, Resistor_SMD:R_0603_1608Metric, F.Cu at (45.5, 67.7)
- added R8: 470, Resistor_SMD:R_0603_1608Metric, F.Cu at (49.0, 109.7)
- added R8: 470, Resistor_SMD:R_0603_1608Metric, F.Cu at (49.0, 88.7)
- added R8: 470, Resistor_SMD:R_0603_1608Metric, F.Cu at (49.0, 67.7)
- added R8: 470, Resistor_SMD:R_0603_1608Metric, F.Cu at (49.0, 46.6)
- added R9: 470, Resistor_SMD:R_0603_1608Metric, F.Cu at (48.6, 95.5)
- added R9: 470, Resistor_SMD:R_0603_1608Metric, F.Cu at (48.6, 74.5)
- added R9: 470, Resistor_SMD:R_0603_1608Metric, F.Cu at (48.6, 53.5)
- added SW1: SW_Push, Button_Switch_SMD:SW_SPST_KMR2, F.Cu at (33.2, 109.2)
- added SW1: SW_Push, Button_Switch_SMD:SW_SPST_KMR2, F.Cu at (33.2, 88.2)
- added SW1: SW_Push, Button_Switch_SMD:SW_SPST_KMR2, F.Cu at (33.2, 67.2)
- added SW2: Reset, Button_Switch_SMD:SW_SPST_KMR2, F.Cu at (64.5, 102.5)
- added SW2: Reset, Button_Switch_SMD:SW_SPST_KMR2, F.Cu at (64.5, 81.5)
- added SW2: Reset, Button_Switch_SMD:SW_SPST_KMR2, F.Cu at (64.5, 60.5)
- added U1: TC1017, Package_TO_SOT_SMD:SOT-353_SC-70-5, F.Cu at (35.0, 95.8)
- added U1: TC1017, Package_TO_SOT_SMD:SOT-353_SC-70-5, F.Cu at (35.0, 74.8)
- added U1: TC1017, Package_TO_SOT_SMD:SOT-353_SC-70-5, F.Cu at (35.0, 53.8)
- added U2: LPC11U35FHI33-501, Package_DFN_QFN:QFN-32-1EP_5x5mm_P0.5mm_EP3.45x3.45mm, F.Cu at (43.2, 103.8)
- added U2: LPC11U35FHI33-501, Package_DFN_QFN:QFN-32-1EP_5x5mm_P0.5mm_EP3.45x3.45mm, F.Cu at (43.2, 82.8)
- added U2: LPC11U35FHI33-501, Package_DFN_QFN:QFN-32-1EP_5x5mm_P0.5mm_EP3.45x3.45mm, F.Cu at (43.2, 61.8)
- added U3: TC1017, Package_TO_SOT_SMD:SOT-353_SC-70-5, F.Cu at (58.0, 99.0)
- added U3: TC1017, Package_TO_SOT_SMD:SOT-353_SC-70-5, F.Cu at (58.0, 78.0)
- added U3: TC1017, Package_TO_SOT_SMD:SOT-353_SC-70-5, F.Cu at (58.0, 57.0)
- added U5: MKW41Z, Package_DFN_QFN:QFN-48-1EP_7x7mm_P0.5mm_EP5.15x5.15mm, F.Cu at (79.5, 102.5)
- added U5: MKW41Z, Package_DFN_QFN:QFN-48-1EP_7x7mm_P0.5mm_EP5.15x5.15mm, F.Cu at (79.5, 81.5)
- added U5: MKW41Z, Package_DFN_QFN:QFN-48-1EP_7x7mm_P0.5mm_EP5.15x5.15mm, F.Cu at (79.5, 60.5)
- added Y1: 12MHz, Crystal:Crystal_SMD_3225-4Pin_3.2x2.5mm, F.Cu at (44.0, 98.0)
- added Y1: 12MHz, Crystal:Crystal_SMD_3225-4Pin_3.2x2.5mm, F.Cu at (44.0, 77.0)
- added Y1: 12MHz, Crystal:Crystal_SMD_3225-4Pin_3.2x2.5mm, F.Cu at (44.0, 56.0)
- added Y2: 32MHz, Crystal:Crystal_SMD_2016-4Pin_2.0x1.6mm, F.Cu at (82.6, 107.7)
- added Y2: 32MHz, Crystal:Crystal_SMD_2016-4Pin_2.0x1.6mm, F.Cu at (82.6, 86.7)
- added Y2: 32MHz, Crystal:Crystal_SMD_2016-4Pin_2.0x1.6mm, F.Cu at (82.6, 65.7)
- added Y3: 32KHz, Crystal:Crystal_SMD_2012-2Pin_2.0x1.2mm, F.Cu at (76.5, 107.5)
- added Y3: 32KHz, Crystal:Crystal_SMD_2012-2Pin_2.0x1.2mm, F.Cu at (76.5, 86.5)
- added Y3: 32KHz, Crystal:Crystal_SMD_2012-2Pin_2.0x1.2mm, F.Cu at (76.5, 65.5)
- added Y3: 32KHz, Crystal:Crystal_SMD_2012-2Pin_2.0x1.2mm, F.Cu at (76.5, 44.5)
- C1, C12, C4, C5, C7, C9: footprint Capacitors_SMD:C_0603 -> Capacitor_SMD:C_0603_1608Metric
- D1, D7, D8: footprint Diodes_SMD:D_SOD-323 -> Diode_SMD:D_SOD-323
- D2, D3, D4, D5, D6: footprint LEDs:LED_0603 -> LED_SMD:LED_0603_1608Metric
- L1: footprint Inductors_SMD:L_0402 -> Inductor_SMD:L_0402_1005Metric
- Q1: footprint TO_SOT_Packages_SMD:SOT-23 -> Package_TO_SOT_SMD:SOT-23
- R1, R10, R11, R13, R14, R15, R16, R3, R4, R5, R6, R7, R9: footprint Resistors_SMD:R_0603 -> Resistor_SMD:R_0603_1608Metric
- SW1, SW2: footprint button:SW_SPST_KMR6 -> Button_Switch_SMD:SW_SPST_KMR2
- U1, U3: footprint TO_SOT_Packages_SMD:SOT-353_SC-70-5 -> Package_TO_SOT_SMD:SOT-353_SC-70-5
- U2: footprint Housings_DFN_QFN:QFN-32-1EP_5x5mm_Pitch0.5mm -> Package_DFN_QFN:QFN-32-1EP_5x5mm_P0.5mm_EP3.45x3.45mm
- U5: footprint Housings_DFN_QFN:QFN-48-1EP_7x7mm_Pitch0.5mm -> Package_DFN_QFN:QFN-48-1EP_7x7mm_P0.5mm_EP5.15x5.15mm
- Y1: footprint Crystals:Crystal_SMD_3225-4pin_3.2x2.5mm -> Crystal:Crystal_SMD_3225-4Pin_3.2x2.5mm
- Y2: footprint Crystals:Crystal_SMD_2016-4pin_2.0x1.6mm -> Crystal:Crystal_SMD_2016-4Pin_2.0x1.6mm
Routing:
- net +3V3: track 509.9 -> 526.6 mm
- net /DIPDAP/TGT_SWCLK: track 150.4 -> 162.8 mm
- net /DIPDAP/TGT_TX: track 182.9 -> 195.1 mm
- net GND: track 433.6 -> 444.1 mm
- net /DIPDAP/TGT_NRESET: track 239.2 -> 249.4 mm
- net /DIPDAP/TGT_SWDIO: track 146.6 -> 156.8 mm
- net /DIPDAP/TGT_RX: track 206.6 -> 216.7 mm
- net Net-(C12-Pad1): track 21.1 -> 22.9 mm
- net Net-(R9-Pad2): track 69.4 -> 70.4 mm
- net /KW41Z/A3: track 110.3 -> 109.3 mm
- net /KW41Z/LED_Green: track 92.0 -> 91.2 mm
- net /KW41Z/A0: track 74.5 -> 75.2 mm
