File: beduino_kw41z/dipdap.sch (KiCad schematic (older format))
At the start: 32 parts

Commit message: Update schematic for new KiCAD version.
Also add some components.
Parts:
- removed C? (x2): 18p, symbol C
- removed SW?: SW_Push, symbol SW_Push
- removed Y?: 12MHz, symbol Crystal
- added SW1: SW_Push, symbol Switch:SW_Push
- added Y1: 12MHz, Crystals:Crystal_SMD_3225-4pin_3.2x2.5mm_HandSoldering, symbol device:Crystal_GND24
- C1, C4: renamed from C?; footprint (none) -> Capacitors_SMD:C_0805_HandSoldering; symbol C -> device:C
- C5, C7: renamed from C?; footprint (none) -> Capacitors_SMD:C_0603_HandSoldering; symbol C -> device:C_Small
- C6, C8: renamed from C?; footprint (none) -> Capacitors_SMD:C_0603_HandSoldering; symbol C -> device:C
- D1: renamed from D?; footprint (none) -> Diodes_SMD:D_SOD-323; symbol D_Schottky -> device:D_Schottky
- D2, D3, D4: renamed from D?; footprint (none) -> LEDs:LED_0603_HandSoldering; symbol LED -> device:LED
- J1: renamed from J?; symbol USB_OTG -> Connector:USB_OTG
- J2: renamed from J?; symbol Conn_01x07 -> Connector:Conn_01x07
- Q1: renamed from Q?; footprint (none) -> TO_SOT_Packages_SMD:SOT-23; symbol Q_PMOS_SGD -> device:Q_PMOS_SGD
- R1, R10, R11, R12, R13, R2, R3, R4, R5, R6, R7, R8, R9: renamed from R?; footprint (none) -> Resistors_SMD:R_0603_HandSoldering; symbol R -> device:R
- U1: renamed from U?; footprint TO_SOT_Packages_SMD:SOT-23-5 -> TO_SOT_Packages_SMD:SOT-23-5_HandSoldering; symbol TC1017 -> beduino_regul:TC1017
- U2: renamed from U?; footprint (none) -> Housings_DFN_QFN:QFN-32-1EP_5x5mm_Pitch0.5mm; symbol LPC11U35FHI33-501 -> beduino_nxp:LPC11U35FHI33-501
Connections:
- wire segments 96 -> 115

Commit message: Small changes in the schematics.
Connections:
- net labels added: USB_N, USB_P, USB_R_N, USB_R_P
- wire segments 115 -> 114
Other:
- moved on the sheet: C4, D1
Changed lines of the file:
@@
 L device:C C4
 U 1 1 5A1F1BE5
-P 3600 2150
-F 0 "C4" H 3715 2196 50  0000 L CNN
-F 1 "10u" H 3715 2105 50  0000 L CNN
-F 2 "Capacitors_SMD:C_0805_HandSoldering" H 3638 2000 50  0001 C CNN
-F 3 "" H 3600 2150 50  0001 C CNN
-	1    3600 2150
+P 3000 2200
+F 0 "C4" H 3115 2246 50  0000 L CNN
+F 1 "10u" H 3115 2155 50  0000 L CNN
+F 2 "Capacitors_SMD:C_0805_HandSoldering" H 3038 2050 50  0001 C CNN
+F 3 "" H 3000 2200 50  0001 C CNN
+	1    3000 2200
 	1    0    0    -1
 $EndComp
@@
 Wire Wire Line
 	2400 2300 2400 2500
-Wire Wire Line
-	3600 2500 3600 2300
 Connection ~ 2400 2500
 Wire Wire Line
@@
 Connection ~ 1050 3950
 NoConn ~ 1350 3700
-Wire Wire Line
-	3600 1700 3600 1900
 Connection ~ 1500 1900
 NoConn ~ 2800 2000
@@
 	1700 1900 1700 2000
 Connection ~ 1700 1900
-Wire Wire Line
-	3200 1900 3600 1900
-Connection ~ 3600 1900
 $Comp
 L device:Q_PMOS_SGD Q1
@@
 Wire Wire Line
 	3000 3100 3200 3100
-Wire Wire Line
-	2100 3600 2250 3600
-Wire Wire Line
-	2100 3500 2600 3500
 $Comp
 L device:R R4
@@
 L device:D_Schottky D1
 U 1 1 5A23E5EA
-P 3050 1900
-F 0 "D1" H 3050 1684 50  0000 C CNN
-F 1 "BAT60A" H 3050 1775 50  0000 C CNN
-F 2 "Diodes_SMD:D_SOD-323" H 3050 1900 50  0001 C CNN
-F 3 "" H 3050 1900 50  0001 C CNN
-	1    3050 1900
+P 3300 1900
+F 0 "D1" H 3300 1684 50  0000 C CNN
+F 1 "BAT60A" H 3300 1775 50  0000 C CNN
+F 2 "Diodes_SMD:D_SOD-323" H 3300 1900 50  0001 C CNN
+F 3 "" H 3300 1900 50  0001 C CNN
+	1    3300 1900
 	-1   0    0    1
 $EndComp
-Wire Wire Line
-	2800 1900 2900 1900
 Wire Wire Line
 	1700 2500 2400 2500
@@
 	2400 2500 2400 2600
 Wire Wire Line
-	2400 2500 3600 2500
+	2400 2500 3000 2500
 Wire Wire Line
 	1900 1900 2000 1900
@@
 	1700 1900 1900 1900
 Wire Wire Line
-	3600 1900 3600 2000
-Wire Wire Line
 	4800 3100 5000 3100
 Wire Wire Line
 	4300 2100 4300 2200
-Wire Wire Line
-	2600 3500 3100 3500
-Wire Wire Line
-	2250 3600 5000 3600
 Wire Wire Line
 	3100 3500 5000 3500
@@
 F 3 "" H 3400 3300 50  0001 C CNN
 	1    3400 3100
-	-1   0    0    -1
+	1    0    0    -1
 $EndComp
 $Comp
@@
 Wire Wire Line
 	4100 5400 4100 5500
+Wire Wire Line
+	2100 3600 5000 3600
+Wire Wire Line
+	2100 3500 3100 3500
+Wire Wire Line
+	3000 1900 3000 2050
+Wire Wire Line
+	3600 1700 3600 1900
+Wire Wire Line
+	2800 1900 3000 1900
+Wire Wire Line
+	3000 1900 3150 1900
+Connection ~ 3000 1900
+Wire Wire Line
+	3450 1900 3600 1900
+Wire Wire Line
+	3000 2350 3000 2500
+Text Label 1500 3500 0    60   ~ 0
+USB_P
+Text Label 1500 3600 0    60   ~ 0
+USB_N
+Text Label 2400 3500 0    60   ~ 0
+USB_R_P
+Text Label 2400 3600 0    60   ~ 0
+USB_R_N
 $EndSCHEMATC

Commit message: Update PCB layout.
The connection between the dipdap and the kw41z-mini is now closed with
a small trace. If the trace is cut, added smd pads simplify the creation
of solder jumpers.
Parts:
- removed Q1: Q_PMOS_SGD, TO_SOT_Packages_SMD:SOT-23, symbol device:Q_PMOS_SGD
- added C2, C3: 18p, Capacitors_SMD:C_0603_HandSoldering, symbol Device:C
- added Q1: Q_PMOS_GSD, TO_SOT_Packages_SMD:SOT-23, symbol Device:Q_PMOS_GSD
- C1, C4, C6, C8: symbol device:C -> Device:C
- C5, C7: symbol device:C_Small -> Device:C
- D1: symbol device:D_Schottky -> Device:D_Schottky
- D2, D3, D4: symbol device:LED -> Device:LED
- J2: symbol Connector:Conn_01x07 -> Connector_Generic:Conn_01x07
- R1, R10, R11, R12, R13, R2, R3, R4, R5, R6, R7, R8, R9: symbol device:R -> Device:R
- SW1: footprint (none) -> Buttons_Switches_SMD:SW_SPST_B3S-1000
- U1: footprint TO_SOT_Packages_SMD:SOT-23-5_HandSoldering -> TO_SOT_Packages_SMD:SOT-353_SC-70-5
- Y1: symbol device:Crystal_GND24 -> Device:Crystal_GND24
Connections:
- net labels removed: USB_N, USB_P, USB_R_N, USB_R_P
- wire segments 114 -> 120
Other:
- moved on the sheet: C4
